File: V2/PCB/CCS.kicad_sch (KiCad schematic)
At the start: 27 parts, among them U901 LM324, U902 CJ431_C3113

Commit message: Schematic "Finished"
Parts:
- removed C111: 220uF, VF_Lib:VF_C_Panasonic_ZA_SizeG_VibrationProof, symbol PGD-Library:C_Polarized_Small
- removed C112: 1uf, Capacitor_SMD:C_0805_2012Metric, symbol PGD-Library:C_Small
- removed C902: 100pF, symbol Device:C_Small
- removed D106: SS54, Diode_SMD:D_SMA, symbol PGD-Library:D_Schottky
- removed JP901: 3.3VRefBridge, symbol Jumper:Jumper_2_Bridged
- removed R118 (x2): 10K, Resistor_SMD:R_0805_2012Metric, symbol PGD-Library:R_Small
- removed R118: 3.16K, Resistor_SMD:R_0805_2012Metric, symbol PGD-Library:R_Small
- removed R901: 11.8K, symbol Device:R_Small
- removed R902: 1.62K, symbol Device:R_Small
- removed R903: 1.1K, symbol Device:R_Small
- removed TP901, TP902: TestPoint, symbol Connector:TestPoint
- removed unit 4 of U901
- removed U902: CJ431_C3113, easyeda2kicad2:SOT-23-3_L2.9-W1.6-P1.90-LS2.8-BR, symbol easyeda2kicad2:CJ431_C3113
- added C801: 100pF, Capacitor_SMD:C_0603_1608Metric, symbol Device:C_Small
- C901: footprint (none) -> Capacitor_SMD:C_0603_1608Metric; JLC Part (none) -> Basic Part; LCSC Part (none) -> C14858
- U901: value LM324 -> LM324DT; footprint (none) -> Package_SO:SOIC-14_3.9x8.7mm_P1.27mm; JLC Part (none) -> Basic Part; LCSC Part (none) -> C71035
- renumbered C112 to C903, C113 to C905, R119 to R904, R119 to R905, R104 to R906, R118 to R907, R118 to R908, R118 to R909, R118 to R913
Connections:
- net OpAmpSupply is gone; now on net OpampPower: C905.2
- net Ref0.4V: now reaches C901.1, R904.2
- net Ref0.4V: now also U901.2 (-); no longer U901.3 (+)
- net at R905.1, U901.6 (-), U901.7: now also C801.2
- net Ref0.25V: now reaches R905.2
- net Ref0.25V: now also U901.3 (+), C801.1; no longer U901.2 (-)
- net +24V renamed OpampPower
Other:
- moved on the sheet: C905
