File: V2/PCB/ADC_ADS1115.kicad_sch (KiCad schematic)
At the start: 8 parts, among them U107 ADS1115IDGS

Commit message: added double plug
Connections:
- net 10VInputConditioner/FilterOut renamed Press0ADC_Filt
- net IDConditioner/FilterOut renamed ID0ADC_Filt
Changed lines of the file:
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@@
+    (effects (font (size 1.27 1.27)) (justify left bottom))
+  )
+  (label "Press0ADC_Filt" (at 116.205 62.23 0) (fields_autoplaced)
+    (effects (font (size 1.27 1.27)) (justify left bottom))
+  )
+  (label "ID0ADC_Filt" (at 114.935 74.93 0) (fields_autoplaced)
     (effects (font (size 1.27 1.27)) (justify left bottom))
   )

Commit message: Schematic "Finished"
Parts:
- renumbered C121 to C401, C117 to C402, C118 to C403, C119 to C404, FB102 to FB401, R115 to R401, R117 to R402, U107 to U401
Connections:
- net 10VInputConditioner1/FilterOut renamed Aux1
- net ID0ADC_Filt renamed Press1ADC_Filt
- net IDConditioner1/FilterOut renamed Aux2
Other:
- removed sheet IDConditioner
- removed sheet IDConditioner1

Commit message: PCB layout first pass
Connections:
- net 3.3vADCSupply: now reaches C402.1, C403.2, C404.2, FB401.2, U401.8 (VDD)
Changed lines of the file:
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@@
+    (effects (font (size 1.27 1.27)) (justify left bottom))
+  )
+  (label "3.3vADCSupply" (at 192.405 66.675 0) (fields_autoplaced)
     (effects (font (size 1.27 1.27)) (justify left bottom))
   )
@@
     )
   )
+  (sheet (at 72.39 72.39) (size 19.05 3.81)
+    (stroke (width 0.1524) (type solid))
+    (fill (color 0 0 0 0.0000))
+    (property "Sheetname" "10VInputConditioner" (at 73.66 71.12 0)
+      (effects (font (size 1.27 1.27)) (justify left bottom))
+    )
+    (property "Sheetfile" "10VInputConditioner.kicad_sch" (at 72.39 76.7846 0)
+      (effects (font (size 1.27 1.27)) (justify left top) hide)
+    )
+    (pin "FilterOut" input (at 91.44 74.295 0)
+      (effects (font (size 1.27 1.27)) (justify right))
+    )
+    (pin "FilterIn" input (at 72.39 74.295 180)
+      (effects (font (size 1.27 1.27)) (justify left))
+    )
+    (instances
+      (project "PiraniGaugeDisplay"
+        (path "/43dd4952-cc68-4687-8eb3-b9ec0d7c6e3f/7c57b138-c155-412b-ab67-530ba4c17690" (page "5"))
+      )
+    )
+  )
   (sheet (at 72.39 59.69) (size 19.05 3.81)
     (stroke (width 0.1524) (type solid))
     (fill (color 0 0 0 0.0000))
-    (property "Sheetname" "10VInputConditioner" (at 73.66 58.42 0)
+    (property "Sheetname" "10VInputConditioner1" (at 72.39 59.055 0)
       (effects (font (size 1.27 1.27)) (justify left bottom))
     )
@@
       (effects (font (size 1.27 1.27)) (justify left))
     )
-    (instances
-      (project "PiraniGaugeDisplay"
-        (path "/43dd4952-cc68-4687-8eb3-b9ec0d7c6e3f/7c57b138-c155-412b-ab67-530ba4c17690" (page "5"))
-      )
-    )
-  )
-  (sheet (at 72.39 72.39) (size 19.05 3.81)
-    (stroke (width 0.1524) (type solid))
-    (fill (color 0 0 0 0.0000))
-    (property "Sheetname" "10VInputConditioner1" (at 72.39 71.755 0)
-      (effects (font (size 1.27 1.27)) (justify left bottom))
-    )
-    (property "Sheetfile" "10VInputConditioner.kicad_sch" (at 72.39 76.7846 0)
-      (effects (font (size 1.27 1.27)) (justify left top) hide)
-    )
-    (pin "FilterOut" input (at 91.44 74.295 0)
-      (effects (font (size 1.27 1.27)) (justify right))
-    )
-    (pin "FilterIn" input (at 72.39 74.295 180)
-      (effects (font (size 1.27 1.27)) (justify left))
-    )
