File: V2/PCB/CCSV2.kicad_sch (KiCad schematic)
At the start: 7 parts, among them U1601 LM334M

Commit message: PCB layout first pass
Connections:
- new net: U1601.5, U1601.8
Changed lines of the file:
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@@
       (effects (font (size 1.27 1.27)) (justify right))
     )
-    (property "Footprint" "Package_SO:SOIC-8_3.9x4.9mm_P1.27mm" (at 132.715 90.17 0)
+    (property "Footprint" "Package_SO:SOIC-8_3.9x4.9mm_P1.27mm" (at 135.255 99.06 0)
       (effects (font (size 1.27 1.27) italic) (justify left) hide)
     )
-    (property "Datasheet" "http://www.ti.com/lit/ds/symlink/lm134.pdf" (at 132.08 86.36 0)
+    (property "Datasheet" "http://www.ti.com/lit/ds/symlink/lm134.pdf" (at 131.445 71.755 0)
       (effects (font (size 1.27 1.27) italic) hide)
     )
@@
     (pin "3")
     (pin "4")
+    (pin "5")
     (pin "6")
     (pin "7")
+    (pin "8")
     (instances
       (project "PiraniGaugeDisplay"
