File: V2/PCB/DualExternalConnector.kicad_sch (KiCad schematic)
At the start: 4 parts, among them J1003 Conn_02x04_Counter_Clockwise, J103 RJ45, J105 DA15_Plug

Commit message: Schematic "Finished"
Parts:
- added C1001, C1002: 1uf, Capacitor_SMD:C_0805_2012Metric, symbol PGD-Library:C_Small
- added D1001: SMAJ30CA, Diode_SMD:D_SMA, symbol PGD-Library:D_TVS
- added R1001, R1002: 4K7, Resistor_SMD:R_0805_2012Metric, symbol PGD-Library:R_Small
- added R1003, R1004: 4k7, Resistor_SMD:R_0402_1005Metric, symbol PGD-Library:R_Small
- J1002: renamed from J1003; footprint (none) -> Connector_PinHeader_2.54mm:PinHeader_2x04_P2.54mm_Vertical
- J1003: renamed from J105; footprint Connector_Dsub:DSUB-15_Male_Horizontal_P2.77x2.84mm_EdgePinOffset4.94mm_Housed_MountingHolesOffset7.48mm -> easyeda2kicad2:DSUB-TH_Z-SUBDRBM602A002; JLC Part (none) -> Extended Part; LCSC Part (none) -> C235810; Mfg Part (none) -> DSUB-TH_Z-SUBDRBM602A002
- TP1001: footprint (none) -> TestPoint:TestPoint_Pad_2.0x2.0mm
- renumbered J103 to J1001
Connections:
- net Relay_Sw_NO is gone; now on net Relay_SP: J1003.4
- net Degas: now also D1001.1 (A1)
- net GND: now also J1003.1, C1001.1, C1002.1, D1001.2 (A2)
- net Relay_SP2 | Rs232Rx: now reaches J1001.6, J1002.2 (Pin_2), J1002.4 (Pin_4)
- net Relay_SP1 | Rs232Tx: now reaches J1001.7, J1002.1 (Pin_1), J1002.3 (Pin_3)
- net +24V renamed PowerIn
- net Relay_A renamed Relay_SP
- net Relay_SP: now also R1002.2, R1004.1; no longer J1003.1
- net Relay_Filament_Status_NO renamed Relay_Filament_Status
- net Relay_Filament_Status: now also R1001.1, R1003.1
- new net +3.3V: R1001.2, R1002.1
- new net Filament_Status/SP2: C1001.2, R1003.2
- new net SP1: C1002.2, R1004.2
Other:
- note added: "Measurement_GND"
- note added: "RelayFilament_GND"
- note added: "Relay_SP_GND"
- note added: "Supply_GND"
- note added: "TX and RX are from the gauges POV here Not Ours, crossover in the parent sheet To keep the pinout matching simpler here"
- moved on the sheet: J1001, J1002, J1003, TP1001

Commit message: PCB layout first pass
Parts:
- J1002: symbol Connector_Generic:Conn_02x04_Counter_Clockwise -> Connector_Generic:Conn_02x04_Odd_Even
- J1003: symbol Connector:DA15_Plug -> Connector:DA15_Plug_MountingHoles
Connections:
- net GND: now also J1003.0 (PAD)
- net RS232_Rx: now also J1002.4 (Pin_4); no longer J1002.7 (Pin_7)
- net RS232_Tx: now also J1002.2 (Pin_2); no longer J1002.8 (Pin_8)
- net Relay_Filament_Status: now also J1002.8 (Pin_8); no longer J1002.5 (Pin_5)
- net Relay_SP1 | Rs232Tx: now also J1002.5 (Pin_5); no longer J1002.3 (Pin_3)
- net Relay_SP2 | Rs232Rx: now also J1002.3 (Pin_3), J1002.7 (Pin_7); no longer J1002.2 (Pin_2), J1002.4 (Pin_4)
Changed lines of the file:
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@@
     (stroke (width 0) (type default))
   )
+  (wire (pts (xy 191.135 106.68) (xy 183.515 106.68))
+    (stroke (width 0) (type default))
+  )
   (wire (pts (xy 182.245 73.025) (xy 186.055 73.025))
     (stroke (width 0) (type default))
@@
     (stroke (width 0) (type default))
   )
+  (wire (pts (xy 183.515 106.68) (xy 183.515 109.22))
+    (stroke (width 0) (type default))
+  )
   (wire (pts (xy 95.25 142.24) (xy 175.895 142.24))
     (stroke (width 0) (type default))
@@
     (stroke (width 0) (type default))
   )
+  (wire (pts (xy 191.135 109.855) (xy 191.135 106.68))
+    (stroke (width 0) (type default))
+  )
   (wire (pts (xy 92.71 107.315) (xy 92.71 129.54))
     (stroke (width 0) (type default))
@@
     (effects (font (size 1.27 1.27)) (justify right))
   )
-  (symbol (lib_id "Connector:DA15_Plug") (at 183.515 132.08 0) (mirror x) (unit 1)
+  (symbol (lib_id "Connector:DA15_Plug_MountingHoles") (at 183.515 132.08 0) (mirror x) (unit 1)
     (in_bom yes) (on_board yes) (dnp no)
     (property "Reference" "J1003" (at 183.1975 108.1151 0)
@@
       (effects (font (size 1.27 1.27)) hide)
     )
-    (property "Datasheet" "https://www.lcsc.com/product-detail/D-Sub-DVI-HDMI-Connectors_Nextron-Nextronics-Engineering-Z-SUBDRBM602A002_C235810.html" (at 183.515 132.08 0)
+    (property "Datasheet" " ~" (at 183.515 132.08 0)
       (effects (font (size 1.27 1.27)) hide)
     )
@@
       (effects (font (size 1.27 1.27)) hide)
     )
+    (pin "0")
     (pin "1")
     (pin "10")
@@
     )
   )
-  (symbol (lib_id "Connector_Generic:Conn_02x04_Counter_Clockwise") (at 95.25 99.695 270) (unit 1)
+  (symbol (lib_id "Connector_Generic:Conn_02x04_Odd_Even") (at 95.25 99.695 270) (unit 1)
     (in_bom yes) (on_board yes) (dnp no)
     (property "Reference" "J1002" (at 92.075 81.28 90)
@@
         )
       )
+    )
+  )
+  (symbol (lib_id "power:GND") (at 191.135 109.855 0) (unit 1)
+    (in_bom yes) (on_board yes) (dnp no) (fields_autoplaced)
+    (property "Reference" "#PWR01006" (at 191.135 116.205 0)
+      (effects (font (size 1.27 1.27)) hide)
+    )
+    (property "Value" "GND" (at 191.135 114.935 0)
+      (effects (font (size 1.27 1.27)))
+    )
+    (property "Footprint" "" (at 191.135 109.855 0)
+      (effects (font (size 1.27 1.27)) hide)
+    )
+    (property "Datasheet" "" (at 191.135 109.855 0)
+      (effects (font (size 1.27 1.27)) hide)
+    )
+    (pin "1")
+    (instances
+      (project "PiraniGaugeDisplay"
+        (path "/43dd4952-cc68-4687-8eb3-b9ec0d7c6e3f/8b3ccaa9-f18e-443a-a99a-510414ad55b9"
+          (reference "#PWR01006") (unit 1)
+        )
+        (path "/43dd4952-cc68-4687-8eb3-b9ec0d7c6e3f/27436e03-7ce1-4a9c-8815-3ff623b3aaa7"
+          (reference "#PWR0706") (unit 1)
+        )
+      )
