File: V2/PCB/HSD.kicad_sch (KiCad schematic)
At the start: 7 parts, among them Q1201 AO3401A, Q1202 AO3401A, Q1203 AO3400A

Commit message: PCB layout first pass
Parts:
- added D102: SS54, Diode_SMD:D_SMA, symbol PGD-Library:D_Schottky
- added D107: LED, LED_SMD:LED_0603_1608Metric, symbol PGD-Library:LED
- added R113: 10K, Resistor_SMD:R_0805_2012Metric, symbol PGD-Library:R_Small
Connections:
- net Drv_Out: now also D102.1 (K), D107.2 (A)
- net GND: now also D102.2 (A), R113.1
- new net: D107.1 (K), R113.2
