File: V2/PCB/Mounting.kicad_sch (KiCad schematic)
At the start: 0 parts

Commit message: PCB layout first pass
Parts:
- added H201, H202, H203, H204: MountingHole, MountingHole:MountingHole_3.2mm_M3, symbol Mechanical:MountingHole
Changed lines of the file:
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@@
 (kicad_sch (version 20230121) (generator eeschema)
   (paper "A4")
+  (symbol (lib_id "Mechanical:MountingHole") (at 38.1 20.32 0) (unit 1)
+    (in_bom yes) (on_board yes) (dnp no) (fields_autoplaced)
+    (property "Reference" "H201" (at 40.64 19.6763 0)
+      (effects (font (size 1.27 1.27)) (justify left))
+    )
+    (property "Value" "MountingHole" (at 40.64 21.5973 0)
+      (effects (font (size 1.27 1.27)) (justify left))
+    )
+    (property "Footprint" "MountingHole:MountingHole_3.2mm_M3" (at 38.1 20.32 0)
+      (effects (font (size 1.27 1.27)) hide)
+    )
+    (property "Datasheet" "~" (at 38.1 20.32 0)
+      (effects (font (size 1.27 1.27)) hide)
+    )
+    (instances
+      (project "PiraniGaugeDisplay"
+        (path "/43dd4952-cc68-4687-8eb3-b9ec0d7c6e3f/fb1654cc-a003-4e40-85a4-ff34d1fb4f4b"
+          (reference "H201") (unit 1)
+        )
+      )
+    )
+  )
+  (symbol (lib_id "Mechanical:MountingHole") (at 38.735 45.72 0) (unit 1)
+    (in_bom yes) (on_board yes) (dnp no) (fields_autoplaced)
+    (property "Reference" "H204" (at 41.275 45.0763 0)
+      (effects (font (size 1.27 1.27)) (justify left))
+    )
+    (property "Value" "MountingHole" (at 41.275 46.9973 0)
+      (effects (font (size 1.27 1.27)) (justify left))
+    )
+    (property "Footprint" "MountingHole:MountingHole_3.2mm_M3" (at 38.735 45.72 0)
+      (effects (font (size 1.27 1.27)) hide)
+    )
+    (property "Datasheet" "~" (at 38.735 45.72 0)
+      (effects (font (size 1.27 1.27)) hide)
+    )
+    (instances
+      (project "PiraniGaugeDisplay"
+        (path "/43dd4952-cc68-4687-8eb3-b9ec0d7c6e3f/fb1654cc-a003-4e40-85a4-ff34d1fb4f4b"
+          (reference "H204") (unit 1)
+        )
+      )
+    )
+  )
+  (symbol (lib_id "Mechanical:MountingHole") (at 37.465 38.1 0) (unit 1)
+    (in_bom yes) (on_board yes) (dnp no) (fields_autoplaced)
+    (property "Reference" "H203" (at 40.005 37.4563 0)
+      (effects (font (size 1.27 1.27)) (justify left))
+    )
+    (property "Value" "MountingHole" (at 40.005 39.3773 0)
+      (effects (font (size 1.27 1.27)) (justify left))
+    )
+    (property "Footprint" "MountingHole:MountingHole_3.2mm_M3" (at 37.465 38.1 0)
+      (effects (font (size 1.27 1.27)) hide)
+    )
+    (property "Datasheet" "~" (at 37.465 38.1 0)
+      (effects (font (size 1.27 1.27)) hide)
+    )
+    (instances
+      (project "PiraniGaugeDisplay"
+        (path "/43dd4952-cc68-4687-8eb3-b9ec0d7c6e3f/fb1654cc-a003-4e40-85a4-ff34d1fb4f4b"
+          (reference "H203") (unit 1)
+        )
+      )
+    )
+  )
+  (symbol (lib_id "Mechanical:MountingHole") (at 39.37 27.94 0) (unit 1)
+    (in_bom yes) (on_board yes) (dnp no) (fields_autoplaced)
+    (property "Reference" "H202" (at 41.91 27.2963 0)
+      (effects (font (size 1.27 1.27)) (justify left))
+    )
+    (property "Value" "MountingHole" (at 41.91 29.2173 0)
+      (effects (font (size 1.27 1.27)) (justify left))
+    )
+    (property "Footprint" "MountingHole:MountingHole_3.2mm_M3" (at 39.37 27.94 0)
+      (effects (font (size 1.27 1.27)) hide)
+    )
+    (property "Datasheet" "~" (at 39.37 27.94 0)
+      (effects (font (size 1.27 1.27)) hide)
+    )
+    (instances
+      (project "PiraniGaugeDisplay"
+        (path "/43dd4952-cc68-4687-8eb3-b9ec0d7c6e3f/fb1654cc-a003-4e40-85a4-ff34d1fb4f4b"
+          (reference "H202") (unit 1)
+        )
+      )
+    )
+  )
 )
