File: V2/PCB/PiraniGaugeDisplay.kicad_pcb (KiCad board)
At the start: 2 copper layers, 87 parts, among them J101 AuxIN, J102 Conn_02x03_Odd_Even, J103 RJ45, U101 AMS1117-3.3, U102 SN75176AD, U103 LM2596S-5, U104 ESP32-S3-WROOM-1(N16R2), U105 SW-SMD_L6.1-W3.5-LS8.0, U106 SW-SMD_L6.1-W3.5-LS8.0, U401 ADS1115IDGS

Commit message: Schematic "Finished"
Parts:
- removed C405: 47uF, PVG2-Library:C_1206_3216Metric
- removed C801: 10uF, PVG2-Library:C_1206_3216Metric
- removed F101: SF-1206F050-2, PVG2-Library:Fuse_1206_3216Metric
- removed FB101: 300m, PVG2-Library:R_0805_2012Metric
- added C1001: 1uf, Capacitor_SMD:C_0805_2012Metric, F.Cu at (179.5, 142.5)
- added C1002: 1uf, Capacitor_SMD:C_0805_2012Metric, F.Cu at (179.5, 145.5)
- added C121: 1uf, Capacitor_SMD:C_0805_2012Metric, F.Cu at (172.4, 105.0)
- added C1401: 100nf, Capacitor_SMD:C_0805_2012Metric, F.Cu at (198.3, 40.0)
- added C1402: 1uf, Capacitor_SMD:C_0805_2012Metric, F.Cu at (198.3, 43.0)
- added C1403: 100nf, Capacitor_SMD:C_0805_2012Metric, F.Cu at (198.3, 46.1)
- added C1404: 100nf, Capacitor_SMD:C_0805_2012Metric, F.Cu at (198.3, 49.1)
- added C1405: 100nf, Capacitor_SMD:C_0805_2012Metric, F.Cu at (198.3, 52.1)
- added C402: 47uF, Capacitor_SMD:C_1206_3216Metric, F.Cu at (194.6, 104.4)
- added C702: 1uf, Capacitor_SMD:C_0805_2012Metric, F.Cu at (137.1, 145.5)
- added D1001: SMAJ30CA, Diode_SMD:D_SMA, F.Cu at (181.4, 138.7)
- added D1101: ZMM5V6-M, Diode_SMD:D_MiniMELF, F.Cu at (211.9, 96.4)
- added D112: LED, LED_SMD:LED_0603_1608Metric, F.Cu at (178.6, 57.3)
- added D113: LED, LED_SMD:LED_0603_1608Metric, F.Cu at (178.6, 59.9)
- added D1201: ZMM5V6-M, Diode_SMD:D_MiniMELF, F.Cu at (213.0, 60.0)
- added D1301: ZMM5V6-M, Diode_SMD:D_MiniMELF, F.Cu at (213.0, 78.2)
- added D1501: ZMM5V6-M, Diode_SMD:D_MiniMELF, F.Cu at (201.9, 117.0)
- added D1601: 1N4148W, Diode_SMD:D_SOD-123, F.Cu at (194.7, 91.0)
- added D701: SMAJ30CA, Diode_SMD:D_SMA, F.Cu at (138.9, 138.7)
- added D801: 1N4148W, Diode_SMD:D_SOD-123, F.Cu at (194.7, 72.8)
- added D901: ZMM5V6-M, Diode_SMD:D_MiniMELF, F.Cu at (201.9, 145.7)
- added FH101: FH1-200CK-B, easyeda2kicad2:FUSE-TH_L24.8-W9.8-P22.60, F.Cu at (156.9, 91.9)
- added J1001: RJ45, SamacSys_Parts:55551621, F.Cu at (156.5, 142.2)
- added J1002: Conn_02x04_Counter_Clockwise, Connector_PinHeader_2.54mm:PinHeader_2x04_P2.54mm_Vertical, F.Cu at (172.4, 138.8)
- added J1003: DA15_Plug, easyeda2kicad2:DSUB-TH_Z-SUBDRBM602A002, F.Cu at (171.6, 119.8)
- added J104: Conn_01x04, easyeda2kicad2:CONN-TH_B4B-XH-A-LF-SN, F.Cu at (136.7, 83.9)
- added J105: Conn_01x04, easyeda2kicad2:CONN-TH_B4B-XH-A-LF-SN, F.Cu at (136.7, 91.0)
- added J106: Conn_01x04, easyeda2kicad2:CONN-TH_B4B-XH-A-LF-SN, F.Cu at (136.7, 98.1)
- added J107: Conn_02x03_Odd_Even, Connector_PinHeader_2.54mm:PinHeader_2x03_P2.54mm_Vertical, F.Cu at (178.9, 40.9)
- added J701: RJ45, SamacSys_Parts:55551621, F.Cu at (114.0, 142.2)
- added J702: Conn_02x04_Counter_Clockwise, Connector_PinHeader_2.54mm:PinHeader_2x04_P2.54mm_Vertical, F.Cu at (130.0, 138.8)
- added J703: DA15_Plug, easyeda2kicad2:DSUB-TH_Z-SUBDRBM602A002, F.Cu at (129.2, 119.8)
- added JP1401: Jumper_2_Bridged, Jumper:SolderJumper-2_P1.3mm_Bridged_Pad1.0x1.5mm, F.Cu at (189.5, 40.3)
- added JP1402: Jumper_2_Bridged, Jumper:SolderJumper-2_P1.3mm_Bridged_Pad1.0x1.5mm, F.Cu at (189.5, 43.9)
- added JP1403: Jumper_2_Bridged, Jumper:SolderJumper-2_P1.3mm_Bridged_Pad1.0x1.5mm, F.Cu at (189.5, 47.4)
- added JP1404: Jumper_2_Bridged, Jumper:SolderJumper-2_P1.3mm_Bridged_Pad1.0x1.5mm, F.Cu at (189.5, 51.0)
- added JP1405: Jumper_2_Bridged, Jumper:SolderJumper-2_P1.3mm_Bridged_Pad1.0x1.5mm, F.Cu at (189.5, 54.5)
- added JP1406: Jumper_2_Bridged, Jumper:SolderJumper-2_P1.3mm_Bridged_Pad1.0x1.5mm, F.Cu at (193.9, 40.3)
- added JP1407: Jumper_2_Bridged, Jumper:SolderJumper-2_P1.3mm_Bridged_Pad1.0x1.5mm, F.Cu at (193.9, 43.9)
- added JP1408: Jumper_2_Bridged, Jumper:SolderJumper-2_P1.3mm_Bridged_Pad1.0x1.5mm, F.Cu at (193.9, 47.4)
- added Q1101: AO3401A, Package_TO_SOT_SMD:SOT-23, F.Cu at (206.3, 96.9)
- added Q1102: AO3401A, Package_TO_SOT_SMD:SOT-23, F.Cu at (206.3, 101.4)
- added Q1103: AO3400A, Package_TO_SOT_SMD:SOT-23, F.Cu at (206.3, 105.8)
- added Q1201: AO3401A, Package_TO_SOT_SMD:SOT-23, F.Cu at (207.3, 60.5)
- added Q1202: AO3401A, Package_TO_SOT_SMD:SOT-23, F.Cu at (207.3, 65.0)
- added Q1203: AO3400A, Package_TO_SOT_SMD:SOT-23, F.Cu at (207.3, 69.4)
- added Q1301: AO3401A, Package_TO_SOT_SMD:SOT-23, F.Cu at (207.3, 78.7)
- added Q1302: AO3401A, Package_TO_SOT_SMD:SOT-23, F.Cu at (207.3, 83.2)
- added Q1303: AO3400A, Package_TO_SOT_SMD:SOT-23, F.Cu at (207.3, 87.6)
- added Q1501: AO3401A, Package_TO_SOT_SMD:SOT-23, F.Cu at (196.2, 117.5)
- added Q1502: AO3401A, Package_TO_SOT_SMD:SOT-23, F.Cu at (196.2, 122.0)
- added Q1503: AO3401A, Package_TO_SOT_SMD:SOT-23, F.Cu at (196.2, 126.4)
- added Q1504: AO3401A, Package_TO_SOT_SMD:SOT-23, F.Cu at (196.2, 130.9)
- added Q1505: AO3401A, Package_TO_SOT_SMD:SOT-23, F.Cu at (196.2, 135.3)
- added Q1506: AO3401A, Package_TO_SOT_SMD:SOT-23, F.Cu at (196.2, 139.8)
- added Q901: AO3401A, Package_TO_SOT_SMD:SOT-23, F.Cu at (196.2, 146.2)
- added Q902: AO3401A, Package_TO_SOT_SMD:SOT-23, F.Cu at (196.2, 150.7)
- added Q903: AO3400A, Package_TO_SOT_SMD:SOT-23, F.Cu at (196.2, 155.1)
- added R1001: 4K7, Resistor_SMD:R_0805_2012Metric, F.Cu at (184.0, 142.5)
- added R1002: 4K7, Resistor_SMD:R_0805_2012Metric, F.Cu at (184.0, 145.4)
- added R1003: 4k7, Resistor_SMD:R_0402_1005Metric, F.Cu at (178.8, 148.0)
- added R1004: 4k7, Resistor_SMD:R_0402_1005Metric, F.Cu at (178.8, 150.0)
- added R1101: 3K6, Resistor_SMD:R_0805_2012Metric, F.Cu at (210.9, 99.5)
- added R1102: 10K, Resistor_SMD:R_0805_2012Metric, F.Cu at (210.9, 102.5)
- added R1103: 1K, Resistor_SMD:R_0402_1005Metric, F.Cu at (210.2, 104.9)
- added R1201: 3K6, Resistor_SMD:R_0805_2012Metric, F.Cu at (212.0, 63.1)
- added R1202: 10K, Resistor_SMD:R_0805_2012Metric, F.Cu at (212.0, 66.0)
- added R1203: 1K, Resistor_SMD:R_0402_1005Metric, F.Cu at (211.2, 68.5)
- added R122: 4K7, Resistor_SMD:R_0805_2012Metric, F.Cu at (154.6, 81.9)
- added R123: 4K7, Resistor_SMD:R_0805_2012Metric, F.Cu at (154.6, 84.9)
- added R124: 4K7, Resistor_SMD:R_0805_2012Metric, F.Cu at (159.0, 67.2)
- added R125: 10K, Resistor_SMD:R_0805_2012Metric, F.Cu at (159.0, 70.1)
- added R126: 3K, Resistor_SMD:R_0805_2012Metric, F.Cu at (159.0, 73.1)
- added R127: 100K, Resistor_SMD:R_0805_2012Metric, F.Cu at (159.0, 76.0)
- added R1301: 3K6, Resistor_SMD:R_0805_2012Metric, F.Cu at (212.0, 81.3)
- added R1302: 10K, Resistor_SMD:R_0805_2012Metric, F.Cu at (212.0, 84.2)
- added R1303: 1K, Resistor_SMD:R_0402_1005Metric, F.Cu at (211.2, 86.7)
- added R1501: 3K6, Resistor_SMD:R_0805_2012Metric, F.Cu at (200.9, 120.1)
- added R1502: 10K, Resistor_SMD:R_0805_2012Metric, F.Cu at (200.9, 123.0)
- added R1601: 3K, Resistor_SMD:R_0805_2012Metric, F.Cu at (189.5, 78.0)
- added R1602: 33K, Resistor_SMD:R_0805_2012Metric, F.Cu at (189.5, 80.9)
- added R1603: 1K2, Resistor_SMD:R_0805_2012Metric, F.Cu at (189.5, 83.9)
- added R1604: 1K, Resistor_SMD:R_0805_2012Metric, F.Cu at (189.5, 86.8)
- added R501: 10K, Resistor_SMD:R_0805_2012Metric, F.Cu at (209.3, 151.9)
- added R502: 2K7, Resistor_SMD:R_0805_2012Metric, F.Cu at (209.3, 154.8)
- added R601: 10K, Resistor_SMD:R_0805_2012Metric, F.Cu at (209.3, 123.2)
- added R602: 2K7, Resistor_SMD:R_0805_2012Metric, F.Cu at (209.3, 126.1)
- added R701: 4K7, Resistor_SMD:R_0805_2012Metric, F.Cu at (141.5, 142.5)
- added R702: 4K7, Resistor_SMD:R_0805_2012Metric, F.Cu at (141.5, 145.4)
- added R703: 4k7, Resistor_SMD:R_0402_1005Metric, F.Cu at (136.3, 148.0)
- added R704: 4k7, Resistor_SMD:R_0402_1005Metric, F.Cu at (136.3, 150.0)
- added R801: 3K, Resistor_SMD:R_0805_2012Metric, F.Cu at (189.5, 59.8)
- added R802: 33K, Resistor_SMD:R_0805_2012Metric, F.Cu at (189.5, 62.7)
- added R803: 1K2, Resistor_SMD:R_0805_2012Metric, F.Cu at (189.5, 65.7)
- added R804: 1K, Resistor_SMD:R_0805_2012Metric, F.Cu at (189.5, 68.6)
- added R901: 3K6, Resistor_SMD:R_0805_2012Metric, F.Cu at (200.9, 148.8)
- added R902: 10K, Resistor_SMD:R_0805_2012Metric, F.Cu at (200.9, 151.8)
- added R903: 1K, Resistor_SMD:R_0402_1005Metric, F.Cu at (200.1, 154.2)
- added RV1601: 1K, Potentiometer_THT:Potentiometer_Bourns_3296Y_Vertical, F.Cu at (199.9, 78.4)
- added RV501: 1K, Potentiometer_THT:Potentiometer_Bourns_3296Y_Vertical, F.Cu at (215.2, 145.9)
- added RV601: 1K, Potentiometer_THT:Potentiometer_Bourns_3296Y_Vertical, F.Cu at (215.2, 117.2)
- added RV801: 1K, Potentiometer_THT:Potentiometer_Bourns_3296Y_Vertical, F.Cu at (199.9, 60.2)
- added SW101: TS-1187A-B-A-B, easyeda2kicad:SW-SMD_4P-L5.1-W5.1-P3.70-LS6.5-TL-2, F.Cu at (164.0, 54.4)
- added SW102: TS-1187A-B-A-B, easyeda2kicad:SW-SMD_4P-L5.1-W5.1-P3.70-LS6.5-TL-2, F.Cu at (164.0, 60.7)
- added TP1001: ThreshA, TestPoint:TestPoint_Pad_2.0x2.0mm, F.Cu at (188.2, 143.0)
- added TP111: IO_46, TestPoint:TestPoint_THTPad_1.5x1.5mm_Drill0.7mm, F.Cu at (182.4, 53.6)
- added TP112: IO_8, TestPoint:TestPoint_THTPad_1.5x1.5mm_Drill0.7mm, F.Cu at (182.4, 57.1)
- added TP701: ThreshA, TestPoint:TestPoint_Pad_2.0x2.0mm, F.Cu at (145.8, 143.0)
- added U107: MX25C-7.62-BK01-02P-CU-S-A, easyeda2kicad2:CONN-TH_2P-P7.62_MAX_MX25C-7.62-BK01-02P-CU-S-A, F.Cu at (119.4, 81.8)
- added U108: MX25C-7.62-BK01-02P-CU-S-A, easyeda2kicad2:CONN-TH_2P-P7.62_MAX_MX25C-7.62-BK01-02P-CU-S-A, F.Cu at (119.4, 99.1)
- added U109: ESP32-S3-WROOM-1(N16R2), easyeda2kicad:WIRELM-SMD_ESP32-S3-WROOM-1, F.Cu at (141.3, 55.5)
- added U1601: LM334M, Package_SO:SOIC-8_3.9x4.9mm_P1.27mm, F.Cu at (196.0, 86.1)
- added U3: SP3232EEY-L/TR, easyeda2kicad2:TSSOP-16_L5.0-W4.4-P0.65-LS6.4-BL, F.Cu at (204.2, 42.8)
- added U801: LM334M, Package_SO:SOIC-8_3.9x4.9mm_P1.27mm, F.Cu at (196.0, 67.9)
- C101, C104: value 100nf -> 47uF; footprint PVG2-Library:C_0805_2012Metric -> Capacitor_SMD:C_1206_3216Metric
- C102, C113, C403, C404: footprint PVG2-Library:C_0805_2012Metric -> Capacitor_SMD:C_0805_2012Metric
- C103, C110, C114: value 47uF -> 100nf; footprint PVG2-Library:C_1206_3216Metric -> Capacitor_SMD:C_0805_2012Metric
- C105, C106, C118: value 1uf -> 47uF; footprint PVG2-Library:C_0805_2012Metric -> Capacitor_SMD:C_1206_3216Metric
- C107, C401, C501, C601: footprint PVG2-Library:C_1206_3216Metric -> Capacitor_SMD:C_1206_3216Metric
- C108: value 47uF -> 220uF; footprint PVG2-Library:C_1206_3216Metric -> VF_Lib:VF_C_Panasonic_ZA_SizeG_VibrationProof
- C109, C117: value 47uF -> 1uf; footprint PVG2-Library:C_1206_3216Metric -> Capacitor_SMD:C_0805_2012Metric
- C111: value 220uF -> 47uF; footprint PVG2-Library:VF_C_Panasonic_ZA_SizeG_VibrationProof -> Capacitor_SMD:C_1206_3216Metric
- C112, C120: value 1uf -> 100nf; footprint PVG2-Library:C_0805_2012Metric -> Capacitor_SMD:C_0805_2012Metric
- C115, C701: value 10uF -> 1uf; footprint PVG2-Library:C_1206_3216Metric -> Capacitor_SMD:C_0805_2012Metric
- C116: value 10uF -> 100nf; footprint PVG2-Library:C_1206_3216Metric -> Capacitor_SMD:C_0805_2012Metric
- C119: value 100nf -> 1uf; footprint PVG2-Library:C_0805_2012Metric -> Capacitor_SMD:C_0805_2012Metric
- D101: value 1N5819WS -> SS54; footprint PVG2-Library:D_SOD-323 -> Diode_SMD:D_SMA
- D102: value ZMM3V3-M -> SS54; footprint PVG2-Library:D_MiniMELF -> Diode_SMD:D_SMA
- D103: value ZMM3V3-M -> 1N5819WS; footprint PVG2-Library:D_MiniMELF -> Diode_SMD:D_SOD-323
- D104: value SMF05CT1G -> LED; footprint PVG2-Library:SOT-363_SC-70-6 -> LED_SMD:LED_0603_1608Metric
- D105: value SS54 -> SMAJ30CA; footprint PVG2-Library:D_SMA -> Diode_SMD:D_SMA
- D106: value SS54 -> LED; footprint PVG2-Library:D_SMA -> LED_SMD:LED_0603_1608Metric
- D107: value SMAJ30CA -> LED; footprint PVG2-Library:D_SMA -> LED_SMD:LED_0603_1608Metric
- D108: value MB10S -> ZMM3V3-M; footprint PVG2-Library:TO-269AA -> Diode_SMD:D_MiniMELF
- D109: value LED -> SS54; footprint PVG2-Library:LED_0603_1608Metric -> Diode_SMD:D_SMA
- D110: value LED -> ZMM3V3-M; footprint PVG2-Library:LED_0603_1608Metric -> Diode_SMD:D_MiniMELF
- D111: value LED -> SMF05CT1G; footprint PVG2-Library:LED_0603_1608Metric -> easyeda2kicad:SOT-363_L2.0-W1.3-P0.65-LS2.1-BR
- FB401, R113, R120: footprint PVG2-Library:R_0805_2012Metric -> Resistor_SMD:R_0805_2012Metric
- J101: value AuxIN -> B8B-XH-A (LF)(SN); footprint PVG2-Library:01x02_LargeSolderPadConnector -> easyeda2kicad2:CONN-TH_B8B-XH-A-LF-SN
- J102: value Conn_02x03_Odd_Even -> Conn_01x04; footprint PVG2-Library:PinHeader_2x03_P2.54mm_Vertical -> easyeda2kicad2:CONN-TH_B4B-XH-A-LF-SN
- J103: value RJ45 -> Conn_01x04; footprint PVG2-Library:55551621 -> easyeda2kicad2:CONN-TH_B4B-XH-A-LF-SN
- L101: footprint PVG2-Library:VF_L_MDA_1040 -> VF_Lib:VF_L_MDA_1040
- R101, R102: value 5K6 -> 4K7; footprint PVG2-Library:R_0402_1005Metric -> Resistor_SMD:R_0805_2012Metric
- R103, R121: value 3K -> 4K7; footprint PVG2-Library:R_0805_2012Metric -> Resistor_SMD:R_0805_2012Metric
- R104: value 1K -> 4K7; footprint PVG2-Library:R_0402_1005Metric -> Resistor_SMD:R_0805_2012Metric
- R105: value 100R -> 4K7; footprint PVG2-Library:R_0805_2012Metric -> Resistor_SMD:R_0805_2012Metric
- R106: value 2K -> 4K7; footprint PVG2-Library:R_0402_1005Metric -> Resistor_SMD:R_0805_2012Metric
- R107: value 3K -> 5K6; footprint PVG2-Library:R_0805_2012Metric -> Resistor_SMD:R_0402_1005Metric
- R108: value 8K2 -> 5K6; footprint PVG2-Library:R_0402_1005Metric -> Resistor_SMD:R_0402_1005Metric
- R109: value 4k7 -> 3K3; footprint PVG2-Library:R_0402_1005Metric -> Resistor_SMD:R_0805_2012Metric
- R110: value 8k2 -> 10K; footprint PVG2-Library:R_0402_1005Metric -> Resistor_SMD:R_0805_2012Metric
- R111: value 4k7 -> 4K7; footprint PVG2-Library:R_0402_1005Metric -> Resistor_SMD:R_0805_2012Metric
- R112, R118: value 10K -> 4K7; footprint PVG2-Library:R_0805_2012Metric -> Resistor_SMD:R_0805_2012Metric
- R114: value 10R -> 3K3; footprint PVG2-Library:R_0805_2012Metric -> Resistor_SMD:R_0805_2012Metric
- R115: value 10R -> 10K; footprint PVG2-Library:R_0805_2012Metric -> Resistor_SMD:R_0805_2012Metric
- R116, R117: value 4K7 -> 10K; footprint PVG2-Library:R_0805_2012Metric -> Resistor_SMD:R_0805_2012Metric
- R119: value 100K -> 4K7; footprint PVG2-Library:R_0805_2012Metric -> Resistor_SMD:R_0805_2012Metric
- R401: value 4K7 -> 10R; footprint PVG2-Library:R_0805_2012Metric -> Resistor_SMD:R_0805_2012Metric
- R402: value 10R -> 4K7; footprint PVG2-Library:R_0805_2012Metric -> Resistor_SMD:R_0805_2012Metric
- TP101, TP102, TP105, TP106, TP107, TP108, TP109, TP110: footprint PVG2-Library:TestPoint_Pad_2.0x2.0mm -> TestPoint:TestPoint_Pad_2.0x2.0mm
- TP103: value TP+BAT -> TP+PwrIn; footprint PVG2-Library:TestPoint_Pad_2.0x2.0mm -> TestPoint:TestPoint_Pad_2.0x2.0mm
- TP104: value TP-BAT -> IO_45; footprint PVG2-Library:TestPoint_Pad_2.0x2.0mm -> TestPoint:TestPoint_THTPad_1.5x1.5mm_Drill0.7mm
- U101: value AMS1117-3.3 -> MX25C-7.62-BK01-02P-CU-S-A; footprint PVG2-Library:SOT-223-3_TabPin2 -> easyeda2kicad2:CONN-TH_2P-P7.62_MAX_MX25C-7.62-BK01-02P-CU-S-A
- U102: value SN75176AD -> AMS1117-3.3; footprint PVG2-Library:SOIC-8_3.9x4.9mm_P1.27mm -> Package_TO_SOT_SMD:SOT-223-3_TabPin2
- U103: footprint PVG2-Library:TO-263-5_TabPin3 -> Package_TO_SOT_SMD:TO-263-5_TabPin3
- U104: value ESP32-S3-WROOM-1(N16R2) -> MAX6675ISA+T; footprint PVG2-Library:WIRELM-SMD_ESP32-S3-WROOM-1 -> easyeda2kicad2:SOIC-8_L5.0-W4.0-P1.27-LS6.0-BL
- U105: value SW-SMD_L6.1-W3.5-LS8.0 -> MX25C-7.62-BK01-02P-CU-S-A; footprint PVG2-Library:SW-SMD_L6.1-W3.5-LS8.0 -> easyeda2kicad2:CONN-TH_2P-P7.62_MAX_MX25C-7.62-BK01-02P-CU-S-A
- U106: value SW-SMD_L6.1-W3.5-LS8.0 -> MAX6675ISA+T; footprint PVG2-Library:SW-SMD_L6.1-W3.5-LS8.0 -> easyeda2kicad2:SOIC-8_L5.0-W4.0-P1.27-LS6.0-BL
- U401: footprint PVG2-Library:TSSOP-10_3x3mm_P0.5mm -> Package_SO:TSSOP-10_3x3mm_P0.5mm
- USBC101: footprint PVG2-Library:USB-C-SMD_TYPE-C-USB-18 -> easyeda2kicad:USB-C-SMD_TYPE-C-USB-18
- moved C501 93.1 mm to (214.3, 152.1)
- moved C403 84.4 mm to (199.6, 100.8)
- moved C404 84.4 mm to (199.6, 103.8)
- moved U401 84.4 mm to (195.2, 97.0)
- moved C401 84.4 mm to (194.6, 101.0)
- moved FB401 84.4 mm to (189.5, 96.2)
- moved R401 84.4 mm to (189.5, 99.1)
- moved R402 84.4 mm to (189.5, 102.1)
- moved C601 83.5 mm to (214.3, 123.4)
- moved D111 73.7 mm to (182.5, 60.5)
- moved D104 72.1 mm to (178.6, 49.5)
- moved D108 69.6 mm to (177.8, 107.4)
- moved D101 69.0 mm to (155.4, 40.8)
- moved U104 63.3 mm to (174.0, 90.5)
- moved U102 62.5 mm to (179.5, 101.6)
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Connections:
- net /ADC_ADS1115/10VInputConditioner/FilterOut renamed /ADC_ADS1115/Press0ADC_Filt
- C102 pad 2: +3.3V -> +5V
- C104 pad 1: +5V -> GND
- C104 pad 2: GND -> +3.3V
- C105 pad 1: /Aux1_Filt -> GND
- C105 pad 2: GND -> /5vB4Diode
- C106 pad 2: /Aux2_Filt -> /5vB4Diode
- C107 pad 2: +5V -> /5vB4Diode
- C108 pad 1: GND -> +24V
- C108 pad 2: /5vB4Diode -> GND
- C109 pad 2: /5vB4Diode -> +24V
- C110 pad 2: /5vB4Diode -> +24V
- C111 pad 1: +24V -> GND
- C111 pad 2: GND -> /5vB4Diode
- C112 pad 2: +24V -> +3.3V
- C113 pad 2: +24V -> +3.3V
- C114 pad 2: /5vB4Diode -> +3.3V
- C115 pad 1: Net-(D108-+) -> /Aux1_Filt
- C116 pad 1: +24V -> GND
- C116 pad 2: GND -> +3.3V
- C117 pad 2: +3.3V -> /Aux2_Filt
- C118 pad 1: +3.3V -> GND
- C118 pad 2: GND -> +3.3V
- C120 pad 1: GND -> +3.3V
- C120 pad 2: /ESP_EN -> GND
- C601 pad 1: /ADC_ADS1115/10VInputConditioner1/FilterOut -> /ADC_ADS1115/Press1ADC_Filt
- C701 pad 1: /ADC_ADS1115/IDConditioner/FilterOut -> GND
- C701 pad 2: GND -> /DualExternalConnector1/Filament_Status/SP2
- D101 pad 2: Net-(D101-A) -> /5vB4Diode
- D102 pad 1: /Aux1_Filt -> /5vSwitchingNode
- D103 pad 1: /Aux2_Filt -> +5V
- D103 pad 2: GND -> Net-(D103-A)
- D104 pad 1: unconnected-(D104-Pad1) -> Net-(D104-K)
- D104 pad 2: GND -> +5V
- D105 pad 1: +5V -> /IdealishDiode/Din
- D105 pad 2: /5vB4Diode -> GND
- D106 pad 1: /5vSwitchingNode -> Net-(D106-K)
- D106 pad 2: GND -> +3.3V
- D107 pad 1: Net-(#FLG0103-pwr) -> Net-(D107-K)
- D107 pad 2: -BATT -> +24V
- D108 pad 1: Net-(D108-+) -> /Aux1_Filt
- D109 pad 1: Net-(D109-K) -> /IdealishDiode/Din
- D109 pad 2: +3.3V -> GND
- D110 pad 1: Net-(D110-K) -> /Aux2_Filt
- D110 pad 2: +5V -> GND
- D111 pad 1: Net-(D111-K) -> unconnected-(D111-Pad1)
- D111 pad 2: +24V -> GND
- J101 pad 1: Net-(J101-Pin_1) -> /BT1
- J101 pad 2: Net-(J101-Pin_2) -> /BT2
- J102 pad 1: /ESP_EN -> GND
- J102 pad 3: /ESP_TXD -> /I2C_SCL
- J102 pad 4: GND -> /I2C_SDA
- J103 pad 2: /ADC_ADS1115/Pressure0 -> +3.3V
- J103 pad 3: unconnected-(J103-Pad3) -> /I2C_SCL
- J103 pad 4: unconnected-(J103-Pad4) -> /I2C_SDA
- R101 pad 1: Net-(USBC101-CC2) -> +3.3V
- R101 pad 2: GND -> /BT1
- R102 pad 1: GND -> +3.3V
- R102 pad 2: Net-(USBC101-CC1) -> /BT2
- R103 pad 1: /485+ -> +3.3V
- R103 pad 2: /A_FIlt -> /BT3
- R104 pad 1: /Rx_D -> +3.3V
- R104 pad 2: Net-(U102-R) -> /BT4
- R105 pad 1: /B_FIlt -> +3.3V
- R105 pad 2: /A_FIlt -> /BT5
- R106 pad 1: GND -> +3.3V
- R106 pad 2: /Rx_D -> /BT6
- R107 pad 1: /485- -> Net-(USBC101-CC2)
- R107 pad 2: /B_FIlt -> GND
- R108 pad 1: /Aux1_Filt -> GND
- R108 pad 2: GND -> Net-(USBC101-CC1)
- R109 pad 1: Net-(J101-Pin_1) -> /Aux1_Filt
- R109 pad 2: /Aux1_Filt -> GND
- R110 pad 1: /Aux2_Filt -> Net-(R110-Pad1)
- R110 pad 2: GND -> /Aux1_Filt
- R111 pad 1: Net-(J101-Pin_2) -> Net-(D104-K)
- R111 pad 2: /Aux2_Filt -> GND
- R112 pad 1: GND -> Net-(D106-K)
- R112 pad 2: Net-(J101-Pin_2) -> GND
- R113 pad 2: Net-(J101-Pin_1) -> Net-(D107-K)
- R114 pad 1: Net-(F101-Pad1) -> /Aux2_Filt
- R114 pad 2: Net-(#FLG0103-pwr) -> GND
- R115 pad 1: Net-(F101-Pad1) -> Net-(R115-Pad1)
- R115 pad 2: Net-(#FLG0103-pwr) -> /Aux2_Filt
- R116 pad 1: Net-(D109-K) -> GND
- R116 pad 2: GND -> Net-(R115-Pad1)
- R117 pad 1: Net-(D110-K) -> GND
- R117 pad 2: GND -> Net-(R110-Pad1)
- R118 pad 1: GND -> +3.3V
- R118 pad 2: Net-(D111-K) -> Net-(J106-Pin_4)
- R119 pad 1: Net-(U104-IO3) -> +5V
- R119 pad 2: +3.3V -> Net-(J106-Pin_3)
- R120 pad 1: +3.3V -> Net-(J106-Pin_2)
- R120 pad 2: /ESP_EN -> +24V
- R121 pad 1: +3.3V -> /ESP_TXD
- R121 pad 2: /ESP_IO0 -> Net-(D112-A)
- R401 pad 1: Net-(U401-ADDR) -> +3.3V
- R401 pad 2: GND -> Net-(C401-Pad1)
- R402 pad 1: +3.3V -> Net-(U401-ADDR)
- R402 pad 2: Net-(C401-Pad1) -> GND
- TP103 pad 1: +BATT -> /PwrIn
- TP104 pad 1: -BATT -> Net-(U109-IO45)
- U101 pad 1: GND -> Net-(U104-T+)
- U101 pad 2: +3.3V -> Net-(U104-T-)
- U102 pad 1: Net-(U102-R) -> GND
- U102 pad 2: /Tx_EN -> +3.3V
- U102 pad 3: /Tx_EN -> +5V
- U104 pad 2: +3.3V -> Net-(U104-T-)
- U104 pad 3: /ESP_EN -> Net-(U104-T+)
- U104 pad 4: unconnected-(U104-IO4-Pad4) -> +3.3V
- U104 pad 5: unconnected-(U104-IO5-Pad5) -> /SPI_SCK
- U104 pad 6: unconnected-(U104-IO6-Pad6) -> /K_CS1
- U104 pad 7: unconnected-(U104-IO7-Pad7) -> /SPI_SDO
- U105 pad 1: /ESP_IO0 -> Net-(U106-T+)
- U105 pad 2: GND -> Net-(U106-T-)
- U106 pad 2: /ESP_EN -> Net-(U106-T-)
- U401 pad 10: /ADC_ADS1115/SCL -> /I2C_SCL
- U401 pad 5: /ADC_ADS1115/IDConditioner/FilterOut -> /ADC_ADS1115/Press1ADC_Filt
- U401 pad 6: /ADC_ADS1115/10VInputConditioner1/FilterOut -> /Aux1_Filt
- U401 pad 7: /ADC_ADS1115/IDConditioner1/FilterOut -> /Aux2_Filt
- U401 pad 9: /ADC_ADS1115/SDA -> /I2C_SDA
- USBC101 pad A4: Net-(D101-A) -> Net-(D103-A)
- USBC101 pad A9: Net-(D101-A) -> Net-(D103-A)
- USBC101 pad B4: Net-(D101-A) -> Net-(D103-A)
- USBC101 pad B9: Net-(D101-A) -> Net-(D103-A)

Commit message: PCB layout first pass
Parts:
- removed J104, J105: Conn_01x04, easyeda2kicad2:CONN-TH_B4B-XH-A-LF-SN
- removed R109, R114: 3K3, Resistor_SMD:R_0805_2012Metric
- removed R110, R115: 10K, Resistor_SMD:R_0805_2012Metric
- removed TP111: IO_46, TestPoint:TestPoint_THTPad_1.5x1.5mm_Drill0.7mm
- added D1102: LED, LED_SMD:LED_0603_1608Metric, F.Cu at (123.1, 102.3)
- added D1103: SS54, Diode_SMD:D_SMA, F.Cu at (125.3, 105.7)
- added D1202: LED, LED_SMD:LED_0603_1608Metric, F.Cu at (122.7, 45.0)
- added D1203: SS54, Diode_SMD:D_SMA, F.Cu at (125.5, 48.4)
- added D1302: LED, LED_SMD:LED_0603_1608Metric, F.Cu at (123.0, 29.9)
- added D1303: SS54, Diode_SMD:D_SMA, F.Cu at (126.1, 33.3)
- added D902: LED, LED_SMD:LED_0603_1608Metric, F.Cu at (123.1, 117.5)
- added D903: SS54, Diode_SMD:D_SMA, F.Cu at (126.8, 120.8)
- added H201: MountingHole, MountingHole:MountingHole_3.2mm_M3, F.Cu at (27.1, 22.2)
- added H202: MountingHole, MountingHole:MountingHole_3.2mm_M3, F.Cu at (152.1, 22.5)
- added H203: MountingHole, MountingHole:MountingHole_3.2mm_M3, F.Cu at (27.1, 162.2)
- added H204: MountingHole, MountingHole:MountingHole_3.2mm_M3, F.Cu at (154.3, 161.9)
- added J108: Aux1_Iso, Connector_PinHeader_2.54mm:PinHeader_1x02_P2.54mm_Vertical, F.Cu at (102.2, 73.0)
- added J109: Aux2_Iso, Connector_PinHeader_2.54mm:PinHeader_1x02_P2.54mm_Vertical, F.Cu at (94.6, 70.5)
- added R1104: 10K, Resistor_SMD:R_0805_2012Metric, F.Cu at (123.1, 98.7)
- added R1204: 10K, Resistor_SMD:R_0805_2012Metric, F.Cu at (122.7, 41.5)
- added R1304: 10K, Resistor_SMD:R_0805_2012Metric, F.Cu at (123.0, 26.3)
- added R904: 10K, Resistor_SMD:R_0805_2012Metric, F.Cu at (123.1, 113.9)
- added RV101: 1K, Potentiometer_THT:Potentiometer_Bourns_3296Y_Vertical, F.Cu at (102.2, 59.7)
- added RV102: 1K, Potentiometer_THT:Potentiometer_Bourns_3296Y_Vertical, F.Cu at (95.3, 64.8)
- added RV103: 1K, Potentiometer_THT:Potentiometer_Bourns_3296Y_Vertical, F.Cu at (102.2, 41.9)
- added RV104: 1K, Potentiometer_THT:Potentiometer_Bourns_3296Y_Vertical, F.Cu at (95.9, 47.0)
- added TP113: TP_Aux1, TestPoint:TestPoint_THTPad_1.5x1.5mm_Drill0.7mm, F.Cu at (106.0, 70.5)
- added TP114: TP_Aux2, TestPoint:TestPoint_THTPad_1.5x1.5mm_Drill0.7mm, F.Cu at (90.8, 70.5)
- JP1401, JP1402, JP1403, JP1404, JP1405, JP1406, JP1407, JP1408: moved to B.Cu
- moved D106 171.6 mm to (25.7, 129.9)
- moved USBC101 168.0 mm to (26.9, 146.3), turned to -90 degrees
- moved D103 167.5 mm to (33.9, 140.8), turned to 180 degrees
- moved D111 167.4 mm to (37.1, 143.5), turned to 180 degrees
- moved D104 165.8 mm to (26.2, 114.8)
- moved C105 162.8 mm to (31.0, 125.2), turned to 90 degrees
- moved R1501 162.4 mm to (46.3, 70.1)
- moved D1501 160.8 mm to (47.3, 72.7)
- moved D107 160.1 mm to (25.4, 101.3)
- moved Q1503 160.0 mm to (44.1, 76.8), turned to 180 degrees
- moved R1502 159.4 mm to (50.5, 70.1)
- moved C106 157.8 mm to (34.8, 125.2), turned to 90 degrees
- moved Q1502 157.4 mm to (44.1, 81.3), turned to 180 degrees
- moved Q1501 155.4 mm to (44.1, 85.7), turned to 180 degrees
- moved Q1504 154.6 mm to (51.4, 76.8)
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Connections:
- net Net-(R110-Pad1) renamed /Aux1_Raw
- net Net-(R115-Pad1) renamed /Aux2_Raw
- net Net-(U401-VDD) renamed /ADC_ADS1115/3.3vADCSupply
- C115 pad 1: /Aux1_Filt -> Net-(D108-K)
- C117 pad 2: /Aux2_Filt -> Net-(D110-K)
- C501 pad 1: /ADC_ADS1115/Press0ADC_Filt -> /ADC_ADS1115/Press1ADC_Filt
- C601 pad 1: /ADC_ADS1115/Press1ADC_Filt -> /ADC_ADS1115/Press0ADC_Filt
- D108 pad 1: /Aux1_Filt -> Net-(D108-K)
- D110 pad 1: /Aux2_Filt -> Net-(D110-K)
- J1001 pad 3: /Press0ADC_Raw -> /DualExternalConnector/Raw_Analog_Measurement
- J1002 pad 2: /DualExternalConnector/Relay_SP2 | Rs232Rx -> /Rx_D_R1
- J1002 pad 3: /DualExternalConnector/Relay_SP1 | Rs232Tx -> /DualExternalConnector/Relay_SP2 | Rs232Rx
- J1002 pad 4: /DualExternalConnector/Relay_SP2 | Rs232Rx -> /Tx_D_R1
- J1002 pad 5: /DualExternalConnector/Relay_Filament_Status -> /DualExternalConnector/Relay_SP1 | Rs232Tx
- J1002 pad 7: /Tx_D_R1 -> /DualExternalConnector/Relay_SP2 | Rs232Rx
- J1002 pad 8: /Rx_D_R1 -> /DualExternalConnector/Relay_Filament_Status
- J1003 pad 2: /Press0ADC_Raw -> /DualExternalConnector/Raw_Analog_Measurement
- J101 pad 8: +5V -> GND
- J702 pad 2: /DualExternalConnector1/Relay_SP2 | Rs232Rx -> /DualExternalConnector1/RS232_Tx
- J702 pad 3: /DualExternalConnector1/Relay_SP1 | Rs232Tx -> /DualExternalConnector1/Relay_SP2 | Rs232Rx
- J702 pad 4: /DualExternalConnector1/Relay_SP2 | Rs232Rx -> /DualExternalConnector1/RS232_Rx
- J702 pad 5: /DualExternalConnector1/Relay_Filament_Status -> /DualExternalConnector1/Relay_SP1 | Rs232Tx
- J702 pad 7: /DualExternalConnector1/RS232_Rx -> /DualExternalConnector1/Relay_SP2 | Rs232Rx
- J702 pad 8: /DualExternalConnector1/RS232_Tx -> /DualExternalConnector1/Relay_Filament_Status
- R501 pad 2: /Press0ADC_Raw -> /DualExternalConnector1/Raw_Analog_Measurement
- R502 pad 2: /ADC_ADS1115/Press0ADC_Filt -> /ADC_ADS1115/Press1ADC_Filt
- R601 pad 2: /DualExternalConnector1/Identification -> /DualExternalConnector/Raw_Analog_Measurement
- R602 pad 2: /ADC_ADS1115/Press1ADC_Filt -> /ADC_ADS1115/Press0ADC_Filt
- R804 pad 1: /DualExternalConnector1/Raw_Analog_Measurement -> /DualExternalConnector1/Identification
- RV501 pad 1: /ADC_ADS1115/Press0ADC_Filt -> /ADC_ADS1115/Press1ADC_Filt
- RV501 pad 2: /ADC_ADS1115/Press0ADC_Filt -> /ADC_ADS1115/Press1ADC_Filt
- RV601 pad 1: /ADC_ADS1115/Press1ADC_Filt -> /ADC_ADS1115/Press0ADC_Filt
- RV601 pad 2: /ADC_ADS1115/Press1ADC_Filt -> /ADC_ADS1115/Press0ADC_Filt
- TP104 pad 1: Net-(U109-IO45) -> unconnected-(TP104-Pad1)
- U109 pad 16: Net-(U109-IO46) -> /K_CS2
- U109 pad 17: /SPI_SCK -> /SPI_SDO
- U109 pad 18: /SPI_SDO -> /DualExternalConnector/Identification
- U109 pad 20: /K_CS2 -> /SPI_SCK
- U109 pad 21: /RS232 - TTL/Rx_D2 -> /RS232 - TTL/Rx_D1
- U109 pad 22: /RS232 - TTL/Tx_D2 -> /RS232 - TTL/Tx_D1
- U109 pad 23: /RS232 - TTL/Rx_D1 -> /RS232 - TTL/Tx_D2
- U109 pad 24: /RS232 - TTL/Tx_D1 -> /RS232 - TTL/Rx_D2
- U109 pad 26: Net-(U109-IO45) -> /EC1_SP1
- U109 pad 33: /I2C_SCL -> /HighSideDriver2/Drv_In
- U109 pad 34: /I2C_SDA -> /HighSideDriver3/Drv_In
- U109 pad 35: /EC1_SP1 -> unconnected-(U109-IO42-Pad35)
- U109 pad 38: /HighSideDriver2/Drv_In -> /I2C_SCL
- U109 pad 39: /HighSideDriver3/Drv_In -> /I2C_SDA
- U109 pad 4: /DualExternalConnector1/Raw_Analog_Measurement -> /DualExternalConnector1/Identification
- U109 pad 5: /DualExternalConnector/Identification -> unconnected-(U109-IO5-Pad5)
- U1601 pad 5: (no net) -> unconnected-(U1601-Pad5)
- U1601 pad 8: (no net) -> unconnected-(U1601-Pad8)
- U801 pad 5: (no net) -> unconnected-(U801-Pad5)
- U801 pad 8: (no net) -> unconnected-(U801-Pad8)
Routing:
- net +3.3V: track 0.00 -> 751.0 mm, vias 0 -> 15
- net +24V: track 0.00 -> 458.9 mm, vias 0 -> 3
- net GND: track 0.00 -> 243.6 mm, vias 0 -> 94
- net /I2C_SDA: track 0.00 -> 176.1 mm, vias 0 -> 3
- net /DualExternalConnector1/Identification: track 0.00 -> 172.6 mm, vias 0 -> 3
- net /I2C_SCL: track 0.00 -> 160.8 mm, vias 0 -> 1
- net /DualExternalConnector/Identification: track 0.00 -> 123.6 mm, vias 0 -> 2
- net /DualExternalConnector1/SP1: track 0.00 -> 111.5 mm, vias 0 -> 2
- net /RS232 - TTL/Rx_D1: track 0.00 -> 108.1 mm, vias 0 -> 1
- net /RS232 - TTL/Tx_D1: track 0.00 -> 106.9 mm, vias 0 -> 1
- net /DualExternalConnector1/Filament_Status/SP2: track 0.00 -> 106.3 mm, vias 0 -> 2
- net /RS232 - TTL/Rx_D2: track 0.00 -> 106.3 mm, vias 0 -> 1
- net /RS232 - TTL/Tx_D2: track 0.00 -> 106.0 mm, vias 0 -> 1
- net /HighSideDriver1/Drv_In: track 0.00 -> 104.7 mm, vias 0 -> 2
- net /DualExternalConnector1/PowerIn: track 0.00 -> 103.8 mm
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- added copper zone on F.Cu, net +24V
- added copper zone on B.Cu, net GND
- added copper zone on F.Cu, net GND
- added copper zone on In1.Cu, net GND
- added copper zone on In2.Cu, net GND
Other:
- board outline added: 150 x 150 mm
- copper layers 2 -> 4
- board text added: "0"
- board text added: "1"
