File: V2/PCB/PiraniGaugeDisplay.kicad_sch (KiCad schematic)
At the start: 82 parts, among them J101 AuxIN, J102 Conn_02x03_Odd_Even, J103 Conn_01x02_Pin, J104 Conn_01x02_Pin, U101 AMS1117-3.3, U102 SN75176AD, U103 LM2596S-5, U104 ESP32-S3-WROOM-1(N16R2), U105 SW-SMD_L6.1-W3.5-LS8.0, U106 SW-SMD_L6.1-W3.5-LS8.0, U107 SP3232EEY-L/TR, U108 MAX6675ISA+T

Commit message: Schematic "Finished"
Parts:
- removed C104, C122, C123, C124, C125: 100nf, Capacitor_SMD:C_0805_2012Metric, symbol PGD-Library:C_Small
- removed C115: 10uF, Capacitor_SMD:C_1206_3216Metric, symbol PGD-Library:C_Small
- removed C121: 1uf, Capacitor_SMD:C_0805_2012Metric, symbol PGD-Library:C_Small
- removed D107: SMAJ30CA, Diode_SMD:D_SMA, symbol PGD-Library:D_TVS
- removed D108: MB10S, Package_TO_SOT_SMD:TO-269AA, symbol PGD-Library:D_Bridge_+-AA
- removed F101: SF-1206F050-2, Fuse:Fuse_1206_3216Metric, symbol PGD-Library:Fuse_Small
- removed FB101: 300m, Resistor_SMD:R_0805_2012Metric, symbol PGD-Library:FerriteBead_Small
- removed J101: AuxIN, VF_Lib:01x02_LargeSolderPadConnector, symbol PGD-Library:Conn_01x02_Socket
- removed J103, J104: Conn_01x02_Pin, symbol Connector:Conn_01x02_Pin
- removed R108: 8K2, Resistor_SMD:R_0402_1005Metric, symbol PGD-Library:R_Small
- removed R109, R111: 4k7, Resistor_SMD:R_0402_1005Metric, symbol PGD-Library:R_Small
- removed R114: 10R, Resistor_SMD:R_0805_2012Metric, symbol PGD-Library:R_Small
- removed U102: SN75176AD, Package_SO:SOIC-8_3.9x4.9mm_P1.27mm, symbol PGD-Library:SN75176AD
- removed U105, U106: SW-SMD_L6.1-W3.5-LS8.0, easyeda2kicad:SW-SMD_L6.1-W3.5-LS8.0, symbol easyeda2kicad:GT-TC060A-H025-L1
- removed U107: SP3232EEY-L/TR, easyeda2kicad2:TSSOP-16_L5.0-W4.4-P0.65-LS6.4-BL, symbol easyeda2kicad2:SP3232EEY-L_TR
- added C113, C114: 100nf, Capacitor_SMD:C_0805_2012Metric, symbol PGD-Library:C_Small
- added D105: SMAJ30CA, Diode_SMD:D_SMA, symbol PGD-Library:D_TVS
- added D109: SS54, Diode_SMD:D_SMA, symbol PGD-Library:D_Schottky
- added D112, D113: LED, LED_SMD:LED_0603_1608Metric, symbol PGD-Library:LED
- added FH101: FH1-200CK-B, easyeda2kicad2:FUSE-TH_L24.8-W9.8-P22.60, symbol easyeda2kicad2:FH1-200CK-B
- added J101: B8B-XH-A (LF)(SN), easyeda2kicad2:CONN-TH_B8B-XH-A-LF-SN, symbol easyeda2kicad2:B8B-XH-A(LF)(SN)
- added J102, J103, J104, J105, J106: Conn_01x04, easyeda2kicad2:CONN-TH_B4B-XH-A-LF-SN, symbol Connector_Generic:Conn_01x04
- added R101, R102, R103, R118, R119, R121, R122, R123, R124: 4K7, Resistor_SMD:R_0805_2012Metric, symbol PGD-Library:R_Small
- added R109, R114: 3K3, Resistor_SMD:R_0805_2012Metric, symbol Device:R_Small
- added R120: 10K, Resistor_SMD:R_0805_2012Metric, symbol PGD-Library:R_Small
- added SW101, SW102: TS-1187A-B-A-B, easyeda2kicad:SW-SMD_4P-L5.1-W5.1-P3.70-LS6.5-TL-2, symbol easyeda2kicad:TS-1187A-B-A-B
- added TP111: IO_46, TestPoint:TestPoint_THTPad_1.5x1.5mm_Drill0.7mm, symbol PGD-Library:TestPoint
- added TP112: IO_8, TestPoint:TestPoint_THTPad_1.5x1.5mm_Drill0.7mm, symbol PGD-Library:TestPoint
- added U101, U105, U107, U108: MX25C-7.62-BK01-02P-CU-S-A, easyeda2kicad2:CONN-TH_2P-P7.62_MAX_MX25C-7.62-BK01-02P-CU-S-A, symbol easyeda2kicad2:MX25C-7.62-BK01-02P-CU-S-A
- added U106: MAX6675ISA+T, easyeda2kicad2:SOIC-8_L5.0-W4.0-P1.27-LS6.0-BL, symbol easyeda2kicad2:MAX6675ISA+T
- C116: value 10uF -> 100nf; footprint Capacitor_SMD:C_1206_3216Metric -> Capacitor_SMD:C_0805_2012Metric; LCSC Part C13585 -> C28233
- D1: footprint Package_TO_SOT_SMD:SOT-363_SC-70-6 -> SOT-363_L2.0-W1.3-P0.65-LS2.1-BR
- R104: value 1K -> 4K7; footprint Resistor_SMD:R_0402_1005Metric -> Resistor_SMD:R_0805_2012Metric; LCSC Part C11702 -> C17673
- R105: value 100R -> 4K7; LCSC Part C17408 -> C17673
- R106: value 2K -> 4K7; footprint Resistor_SMD:R_0402_1005Metric -> Resistor_SMD:R_0805_2012Metric; LCSC Part C4109 -> C17673
- R110: value 8k2 -> 10K; footprint Resistor_SMD:R_0402_1005Metric -> Resistor_SMD:R_0805_2012Metric; LCSC Part C25924 -> C17414
- R115: value 10R -> 10K; LCSC Part C17415 -> C17414
- TP103: value TP+BAT -> TP+PwrIn
- TP104: value TP-BAT -> IO_45; footprint TestPoint:TestPoint_Pad_2.0x2.0mm -> TestPoint:TestPoint_THTPad_1.5x1.5mm_Drill0.7mm
- renumbered C107 to C101, C101 to C102, C102 to C103, C103 to C104, C108 to C105, C109 to C106, C110 to C107, C111 to C108, C112 to C109, C113 to C110, C114 to C111, C126 to C112, C105 to C115, C106 to C117, C117 to C118, C118 to C119, C119 to C120, C120 to C121, D105 to D101, D106 to D102, D110 to D104, D109 to D106, D111 to D107, D102 to D108, D103 to D110, J102 to J107, R117 to R111, R116 to R112, R118 to R113, R112 to R116, R113 to R117, R120 to R125, R121 to R126, R119 to R127, U101 to U102, U108 to U104, U104 to U109
Connections:
- net 485+ is gone; now on net +3.3V: R105.1
- net CAN_R is gone; now on an unnamed net: U109.26 (IO45)
- net Tx_D is gone; now on net BT5: U109.10 (IO17)
- net Tx_D1 is gone; now on net BT4: U109.9 (IO16)
- net +24V: now also R120.2; no longer C116.1
- net +3.3V: now also C116.2, R104.1, R106.1, C113.2, C114.2, J101.7, J102.2 (Pin_2), J103.2 (Pin_2), R101.1, R102.1, R103.1, R118.1, R122.1, R123.1, U106.4 (VCC)
- net +5V: now also J101.8, R119.1
- net Aux1_Filt: now also R110.2, R109.1; no longer U109.17 (IO9)
- net Aux2_Filt: now also R115.2, R114.1; no longer R110.1, U109.16 (IO46)
- net ESP_EN: now also SW102.3 (C), SW102.4 (D)
- net ESP_IO0: now also SW101.1 (A), SW101.2 (B)
- net ESP_RXD: now also R124.1
- net ESP_TXD: now also R121.1
- net GND: now also C116.1, C113.1, C114.1, D105.2 (A2), D109.2 (A), D112.1 (K), D113.1 (K), J101., J102.1 (Pin_1), J103.1 (Pin_1), J104.1 (Pin_1), J105.1 (Pin_1), J106.1 (Pin_1), R109.2, R114.2, SW101.3 (C), SW101.4 (D), SW102.1 (A), SW102.2 (B), U106.1 (GND), U107.1; no longer C116.2, R106.1, R110.2
- net SPI_SCK: now also U109.17 (IO9), U106.5 (SCK); no longer U109.18 (IO10)
- net SPI_SDO: now also U109.18 (IO10), U106.7 (SO); no longer U109.20 (IO12)
- net at U104.2 (T-): now also U101.2
- net at U104.3 (T+): now also U101.1
- net BT5: now reaches R105.2
- net BT5: now also J101.5, J104.3 (Pin_3)
- net RS232 - TTL/Rx_D2: now reaches U109.21 (IO13)
- net RS232 - TTL/Tx_D2: now reaches U109.22 (IO14)
- net RS232 - TTL/Rx_D1: now reaches U109.23 (IO21)
- net RS232 - TTL/Tx_D1: now reaches U109.24 (IO47)
- net DualExternalConnector1/Filament_Status/SP2: now reaches U109.28 (IO35)
- net HighSideDriver/Drv_In: now reaches U109.31 (IO38)
- net EC1_SP1: now reaches U109.35 (IO42)
- net HighSideDriver2/Drv_In: now reaches U109.38 (IO2)
- net HighSideDriver3/Drv_In: now reaches U109.39 (IO1)
- net at R117.2: now also R110.1, U108.1
- net at R115.1: now also R116.2, U108.2
- net BT4: now reaches R104.2
- net BT4: now also J101.4, J104.2 (Pin_2)
- net +BATT renamed PwrIn
- net PwrIn: now also FH101.2, U107.2
- net -BATT: no longer names the net of TP104.1
- net ADC_ADS1115/SCL renamed I2C_SCL
- net I2C_SCL: now also J102.3 (Pin_3), J103.3 (Pin_3), R123.2
- net ADC_ADS1115/SDA renamed I2C_SDA
- net I2C_SDA: now also J102.4 (Pin_4), J103.4 (Pin_4), R122.2
- net CAN+: no longer names the net of D1.6
- net CAN-: no longer names the net of D1.5
- net CAN_D renamed EC1_SP2
- net ConstantCurrentSource/CC_Scaled_Out renamed CCSv2/19uAOut
- net ConstantCurrentSource1/CC_Scaled_Out renamed CCSv3/19uAOut
- net K_CS renamed K_CS1
- net Rx_D renamed BT6
- net BT6: now also J101.6, J104.4 (Pin_4); no longer R104.1
- net Rx_D1 renamed BT3
- net BT3: now also J101.3, J105.4 (Pin_4), R103.2
- net Rx_D2 renamed BT1
- net BT1: now also J101.1, J105.2 (Pin_2), R101.2; no longer U109.30 (IO37)
- net Tx_D2 renamed BT2
- net BT2: now also J101.2, J105.3 (Pin_3), R102.2; no longer U109.29 (IO36)
- net Tx_EN: no longer names the net of U109.12 (IO8)
- net Tx_EN: now also TP112.1
- new net: J106.3 (Pin_3), R119.2
- new net: D113.2 (A), R124.2
- new net: D112.2 (A), R121.2
- new net: TP111.1, U109.16 (IO46)
- new net: U105.1, U106.3 (T+)
- new net: U105.2, U106.2 (T-)
- new net: J106.4 (Pin_4), R118.2
- new net: J106.2 (Pin_2), R120.1
- new net DualExternalConnector1/SP1: U109.29 (IO36)
- new net HighSideDriver1/Drv_In: U109.30 (IO37)
- new net IdealishDiode/Din: D105.1 (A1), D109.1 (K), FH101.1
- new net K_CS2: U106.6 (~{CS}), U109.20 (IO12)
- no-connect marks 11 -> 19
Other:
- removed sheet ConstantCurrentSource
- removed sheet ConstantCurrentSource1
- added sheet CCSv2 (CCSV2.kicad_sch)
- added sheet CCSv3 (CCSV2.kicad_sch)
- added sheet HighSideDriver (HSD.kicad_sch)
- added sheet HighSideDriver1 (HSD.kicad_sch)
- added sheet HighSideDriver2 (HSD.kicad_sch)
- added sheet HighSideDriver3 (HSD.kicad_sch)
- added sheet IdealishDiode (IdealishDiode.kicad_sch)
- added sheet RS232 - TTL (rs2322ttl.kicad_sch)
- sheet ADC_ADS1115 ports: added Aux1, Aux2; removed ID0, ID1
- sheet DualExternalConnector ports: added Filament_Status/SP2, PowerIn, SP1; removed Relay_A, Relay_Filament_Status_NO, Relay_Sw_NO
- sheet DualExternalConnector1 ports: added Filament_Status/SP2, PowerIn, SP1; removed Relay_A, Relay_Filament_Status_NO, Relay_Sw_NO
- note added: "+5 and 3.3 here for future utility"
- note added: "After initial prog these are used for status display"
- note added: "Aux Input 0-10V The over voltage and ESD diode will probably leak at the top end of that range"
- note added: "Button interface"
- note added: "Hard Pullup"
- note added: "Reverse Polarity Crowbar"
- note added: "TODO Set the DB15 plug to being a real part (lcsc etc) Fix floating opamps"
- note added: "Thermocouples"
- note removed: "0.5A Fuse Fast Blow"
- note removed: "5V IC, watch for level shifts"
- note removed: "Aux Input"
- note removed: "Diode bridge creates 0.6v Gnd offset"
- note removed: "RS485(ish)"
- note removed: "Res ~90Hz"
- note removed: "TODO Change input resistance for 1.5A minimum for power for gauges Add ADC Change boot/reset switches to JLC basic lib parts Set the DB15 plug to being a real part (lcsc etc)"
- moved on the sheet: C112, C118, C119, C120, D104, D106, D107, R111, R112, R113, R125, R126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

Commit message: PCB layout first pass
Parts:
- removed J104, J105: Conn_01x04, easyeda2kicad2:CONN-TH_B4B-XH-A-LF-SN, symbol Connector_Generic:Conn_01x04
- removed R109, R114: 3K3, Resistor_SMD:R_0805_2012Metric, symbol Device:R_Small
- removed R110, R115: 10K, Resistor_SMD:R_0805_2012Metric, symbol PGD-Library:R_Small
- removed TP111: IO_46, TestPoint:TestPoint_THTPad_1.5x1.5mm_Drill0.7mm, symbol PGD-Library:TestPoint
- added J108: Aux1_Iso, Connector_PinHeader_2.54mm:PinHeader_1x02_P2.54mm_Vertical, symbol Connector:Conn_01x02_Pin
- added J109: Aux2_Iso, Connector_PinHeader_2.54mm:PinHeader_1x02_P2.54mm_Vertical, symbol Connector:Conn_01x02_Pin
- added RV1601 (x4): 1K, Potentiometer_THT:Potentiometer_Bourns_3296Y_Vertical, symbol Device:R_Potentiometer_Trim
- added TP113: TP_Aux1, TestPoint:TestPoint_THTPad_1.5x1.5mm_Drill0.7mm, symbol PGD-Library:TestPoint
- added TP114: TP_Aux2, TestPoint:TestPoint_THTPad_1.5x1.5mm_Drill0.7mm, symbol PGD-Library:TestPoint
Connections:
- net +5V: no longer J101.8
- net Aux1_Filt: now also J108.1 (Pin_1); no longer C115.1, D108.1 (K)
- net Aux2_Filt: now also J109.2 (Pin_2); no longer C117.2, D110.1 (K)
- net CCSv2_I1/19uAOut: now also U109.18 (IO10); no longer U109.5 (IO5)
- net EC1_SP1: now also U109.26 (IO45); no longer U109.35 (IO42)
- net GND: now also J101.8, RV1601.2, RV1601.2; no longer J101.
- net HighSideDriver2/Drv_In: now also U109.33 (IO40); no longer U109.38 (IO2)
- net HighSideDriver3/Drv_In: now also U109.34 (IO41); no longer U109.39 (IO1)
- net I2C_SCL: now also U109.38 (IO2); no longer U109.33 (IO40)
- net I2C_SDA: now also U109.39 (IO1); no longer U109.34 (IO41)
- net K_CS2: now also U109.16 (IO46); no longer U109.20 (IO12)
- net RS232 - TTL/Rx_D1: now also U109.21 (IO13); no longer U109.23 (IO21)
- net RS232 - TTL/Rx_D2: now also U109.24 (IO47); no longer U109.21 (IO13)
- net RS232 - TTL/Tx_D1: now also U109.22 (IO14); no longer U109.24 (IO47)
- net RS232 - TTL/Tx_D2: now also U109.23 (IO21); no longer U109.22 (IO14)
- net SPI_SCK: now also U109.20 (IO12); no longer U109.17 (IO9)
- net SPI_SDO: now also U109.17 (IO9); no longer U109.18 (IO10)
- net Aux1_Raw: now reaches R117.2, U108.1
- net Aux1_Raw: now also RV1601.1
- net Aux2_Raw: now reaches R116.2, U108.2
- net Aux2_Raw: now also RV1601.3
- net at TP104.1: no longer U109.26 (IO45)
- new net: C115.1, D108.1 (K), J108.2 (Pin_2), RV1601.1, RV1601.2, TP113.1
- new net: C117.2, D110.1 (K), J109.1 (Pin_1), RV1601.2, RV1601.3, TP114.1
- no-connect marks 19 -> 24
Other:
- sheet CCSv2 renamed CCSv2_I1
- sheet CCSv3 renamed CCSv2_I0
- note added: "0"
- note added: "1"
- note added: "3.3v here for future utility"
- note added: "Aux Input adjustable divider The over voltage and ESD diode will probably leak at the top end of the range"
- note added: "Due to skill and dexterity these are reversed top to bottom from the schematic to the PCB, A1 winning"
- note removed: "+5 and 3.3 here for future utility"
- note removed: "Aux Input 0-10V The over voltage and ESD diode will probably leak at the top end of that range"
- moved on the sheet: R116, R117, R122, R123, TP104, U108
